Commit message: 0

File: my_robot_ws/build/my_car_bot/urdf/robot.urdf.xacro (robot description, xacro)
@@ -1 +1 @@
-/media/a-qassem/01DBC69DA6BBEB20/FCIS/ROB/Robotics-task/my_robot_ws/src/my_car_bot/urdf/robot.urdf.xacro
+/media/a-qassem/01DBC69DA6BBEB20/FCIS/ROB/task-for-everyone/Robotics-task/my_robot_ws/src/my_car_bot/urdf/robot.urdf.xacro

File: my_robot_ws/install/my_car_bot/share/my_car_bot/urdf/robot.urdf.xacro (robot description, xacro)
@@ -1 +1 @@
-/media/a-qassem/01DBC69DA6BBEB20/FCIS/ROB/Robotics-task/my_robot_ws/build/my_car_bot/urdf/robot.urdf.xacro
+/media/a-qassem/01DBC69DA6BBEB20/FCIS/ROB/task-for-everyone/Robotics-task/my_robot_ws/build/my_car_bot/urdf/robot.urdf.xacro

File: my_robot_ws/src/my_car_bot/urdf/robot.urdf.xacro (robot description, xacro)
@@ -1,17 +1,27 @@
 <robot xmlns:xacro="http://www.ros.org/wiki/xacro" name="car_bot">
-    <!-- Robot Material Colors -->
-    <material name="white">
-        <color rgba="1 1 1 1"/>
-    </material>
-    <material name="orange">
-        <color rgba="1 0.5 0 1"/>
-    </material>
-    <material name="black">
-        <color rgba="0.1 0.1 0.1 1"/>
-    </material>
-    <material name="blue_glow">
-        <color rgba="0.0 0.8 1.0 1"/>
-    </material>
-    <!-- Base Link (Chassis) -->
+    <!-- ======================= -->
+    <!-- PURPLE EXPLORER MATERIALS -->
+    <!-- ======================= -->
+    <!-- Main body - vibrant purple like reference -->
+    <material name="body_purple">
+        <color rgba="0.4 0.1 0.7 1"/>
+    </material>
+    <!-- Darker purple for accents -->
+    <material name="accent_purple">
+        <color rgba="0.3 0.05 0.5 1"/>
+    </material>
+    <!-- Gray wheels with metallic look -->
+    <material name="wheel_gray">
+        <color rgba="0.4 0.4 0.45 1"/>
+    </material>
+    <!-- Light gray for rims -->
+    <material name="rim_silver">
+        <color rgba="0.7 0.7 0.75 1"/>
+    </material>
+    <!-- Dark sensor housing -->
+    <material name="sensor_dark">
+        <color rgba="0.15 0.15 0.2 1"/>
+    </material>
+    <!-- Base Link (Virtual) -->
     <link name="base_link">
     </link>
@@ -20,70 +30,131 @@
         <parent link="base_link"/>
         <child link="chassis"/>
-        <origin xyz="0 0 0.28"/>
+        <origin xyz="0 0 0.15"/>
     </joint>
     <link name="chassis">
-        <!-- Main Sphere Body -->
-        <visual>
+        <!-- Main Box Body - Purple -->
+        <visual>
+            <origin xyz="0 0 0.05" rpy="0 0 0"/>
+            <geometry>
+                <box size="0.5 0.35 0.18"/>
+            </geometry>
+            <material name="body_purple"/>
+        </visual>
+        <collision>
+            <origin xyz="0 0 0.05" rpy="0 0 0"/>
+            <geometry>
+                <box size="0.5 0.35 0.18"/>
+            </geometry>
+        </collision>
+        <!-- Top Platform / Equipment Deck -->
+        <visual>
+            <origin xyz="-0.05 0 0.16" rpy="0 0 0"/>
+            <geometry>
+                <box size="0.35 0.3 0.04"/>
+            </geometry>
+            <material name="body_purple"/>
+        </visual>
+        <!-- Front Bumper Section (slightly extended) -->
+        <visual>
+            <origin xyz="0.22 0 -0.02" rpy="0 0 0"/>
+            <geometry>
+                <box size="0.1 0.38 0.1"/>
+            </geometry>
+            <material name="accent_purple"/>
+        </visual>
+        <!-- Rear Bumper Section -->
+        <visual>
+            <origin xyz="-0.22 0 -0.02" rpy="0 0 0"/>
+            <geometry>
+                <box size="0.1 0.38 0.1"/>
+            </geometry>
+            <material name="accent_purple"/>
+        </visual>
+        <!-- Side Rails (Left) -->
+        <visual>
+            <origin xyz="0 0.175 0.02" rpy="0 0 0"/>
+            <geometry>
+                <box size="0.4 0.02 0.12"/>
+            </geometry>
+            <material name="accent_purple"/>
+        </visual>
+        <!-- Side Rails (Right) -->
+        <visual>
+            <origin xyz="0 -0.175 0.02" rpy="0 0 0"/>
+            <geometry>
+                <box size="0.4 0.02 0.12"/>
+            </geometry>
+            <material name="accent_purple"/>
+        </visual>
+        <!-- Control Box on Top -->
+        <visual>
+            <origin xyz="-0.12 0.08 0.2" rpy="0 0 0"/>
+            <geometry>
+                <box size="0.08 0.1 0.06"/>
+            </geometry>
+            <material name="sensor_dark"/>
+        </visual>
+        <!-- Antenna Mount -->
+        <visual>
+            <origin xyz="-0.2 -0.1 0.22" rpy="0 0 0"/>
+            <geometry>
+                <cylinder radius="0.015" length="0.08"/>
+            </geometry>
+            <material name="sensor_dark"/>
+        </visual>
+        <!-- Antenna Stick -->
+        <visual>
+            <origin xyz="-0.2 -0.1 0.35" rpy="0 0 0"/>
+            <geometry>
+                <cylinder radius="0.005" length="0.2"/>
+            </geometry>
+            <material name="sensor_dark"/>
+        </visual>
+        <inertial>
             <origin xyz="0 0 0" rpy="0 0 0"/>
-            <geometry>
-                <sphere radius="0.25"/>
-            </geometry>
-            <material name="white"/>
-        </visual>
-        <collision>
-            <origin xyz="0 0 0" rpy="0 0 0"/>
-            <geometry>
-                <sphere radius="0.25"/>
-            </geometry>
-        </collision>
-        <!-- Orange Stripe/Detail -->
-        <visual>
-            <origin xyz="0 0 0" rpy="0 0 0"/>
-            <geometry>
-                <cylinder radius="0.252" length="0.05"/>
-            </geometry>
-            <material name="orange"/>
-        </visual>
-        <!-- The "Eye" -->
-        <visual>
-            <origin xyz="0.22 0 0.05" rpy="0 1.57 0"/>
-            <geometry>
-                <cylinder radius="0.08" length="0.05"/>
-            </geometry>
-            <material name="black"/>
-        </visual>
-        <visual>
-            <origin xyz="0.25 0 0.05" rpy="0 1.57 0"/>
-            <geometry>
-                <cylinder radius="0.06" length="0.01"/>
-            </geometry>
-            <material name="blue_glow"/>
-        </visual>
-        <inertial>
-            <origin xyz="0 0 -0.15" rpy="0 0 0"/>
-            <mass value="5.0"/>
-            <inertia ixx="0.1" ixy="0.0" ixz="0.0" iyy="0.1" iyz="0.0" izz="0.1"/>
+            <mass value="12.0"/>
+            <inertia ixx="0.25" ixy="0.0" ixz="0.0" iyy="0.25" iyz="0.0" izz="0.25"/>
         </inertial>
     </link>
-    <!-- LIDAR (Hidden inside or on top? Let's put it on top like a small antenna) -->
+    <gazebo reference="chassis">
+        <material>Gazebo/Purple</material>
+    </gazebo>
+    <!-- Lidar Tower Mount -->
     <joint name="laser_joint" type="fixed">
         <parent link="chassis"/>
         <child link="laser_frame"/>
-        <origin xyz="0 0 0.26" rpy="0 0 0"/>
+        <origin xyz="0.05 0 0.25" rpy="0 0 0"/>
     </joint>
     <link name="laser_frame">
-        <visual>
-            <geometry>
-                <cylinder radius="0.03" length="0.04"/>
-            </geometry>
-            <material name="black"/>
+        <!-- Pillar Base -->
+        <visual>
+            <origin xyz="0 0 -0.05" rpy="0 0 0"/>
+            <geometry>
+                 <cylinder radius="0.035" length="0.08"/>
+            </geometry>
+            <material name="sensor_dark"/>
+        </visual>
+        <!-- Sensor Head (Cylinder) -->
+        <visual>
+            <geometry>
+                <cylinder radius="0.045" length="0.05"/>
+            </geometry>
+            <material name="sensor_dark"/>
+        </visual>
+        <!-- Top Cap -->
+        <visual>
+            <origin xyz="0 0 0.03" rpy="0 0 0"/>
+            <geometry>
+                <cylinder radius="0.04" length="0.01"/>
+            </geometry>
+            <material name="rim_silver"/>
         </visual>
         <collision>
             <geometry>
-                <cylinder radius="0.03" length="0.04"/>
+                <cylinder radius="0.045" length="0.05"/>
             </geometry>
         </collision>
         <inertial>
-            <mass value="0.1"/>
+            <mass value="0.2"/>
             <inertia ixx="0.001" ixy="0" ixz="0" iyy="0.001" iyz="0" izz="0.001"/>
         </inertial>
@@ -93,5 +164,5 @@
             <pose>0 0 0 0 0 0</pose>
             <always_on>true</always_on>
-            <visualize>true</visualize>
+            <visualize>false</visualize>
             <update_rate>10</update_rate>
             <topic>scan</topic>
@@ -113,18 +184,36 @@
         </sensor>
     </gazebo>
-    <!-- DRIVE WHEELS (Large Side Wheels) -->
-    <xacro:macro name="drive_wheel" params="prefix y_reflect">
+    <!-- 4 WHEEL SYSTEM -->
+    <!-- Macro for Off-road Wheels like in reference -->
+    <xacro:macro name="explorer_wheel" params="prefix x_pos y_pos friction:=1.0">
         <link name="${prefix}_wheel">
+            <!-- Outer Tire - Gray rubber look -->
             <visual>
                 <origin xyz="0 0 0" rpy="${pi/2} 0 0"/>
                 <geometry>
-                    <cylinder radius="0.12" length="0.05"/>
-                </geometry>
-                <material name="orange"/>
+                    <cylinder radius="0.1" length="0.08"/>
+                </geometry>
+                <material name="wheel_gray"/>
+            </visual>
+            <!-- Inner Rim - Silver -->
+            <visual>
+                <origin xyz="0 0 0" rpy="${pi/2} 0 0"/>
+                <geometry>
+                    <cylinder radius="0.06" length="0.085"/>
+                </geometry>
+                <material name="rim_silver"/>
+            </visual>
+            <!-- Hub Cap -->
+            <visual>
+                <origin xyz="0 0.045 0" rpy="${pi/2} 0 0"/>
+                <geometry>
+                    <cylinder radius="0.03" length="0.01"/>
+                </geometry>
+                <material name="sensor_dark"/>
             </visual>
             <collision>
                 <origin xyz="0 0 0" rpy="${pi/2} 0 0"/>
                 <geometry>
-                    <cylinder radius="0.12" length="0.05"/>
+                    <cylinder radius="0.1" length="0.08"/>
                 </geometry>
             </collision>
@@ -132,5 +221,5 @@
                 <origin xyz="0 0 0" rpy="0 0 0"/>
                 <mass value="2.0"/>
-                <inertia ixx="0.01" ixy="0.0" ixz="0.0" iyy="0.01" iyz="0.0" izz="0.01"/>
+                <inertia ixx="0.02" ixy="0.0" ixz="0.0" iyy="0.02" iyz="0.0" izz="0.02"/>
             </inertial>
         </link>
@@ -138,48 +227,27 @@
             <parent link="base_link"/>
             <child link="${prefix}_wheel"/>
-            <origin xyz="0 ${y_reflect*0.30} 0.12" rpy="0 0 0"/>
+            <origin xyz="${x_pos} ${y_pos} 0.1" rpy="0 0 0"/>
             <axis xyz="0 1 0"/>
         </joint>
         <gazebo reference="${prefix}_wheel">
-            <mu1>1.0</mu1>
-            <mu2>1.0</mu2>
+             <!-- Friction Parameter -->
+            <mu1>${friction}</mu1>
+            <mu2>${friction}</mu2>
+            <material>Gazebo/Grey</material>
         </gazebo>
     </xacro:macro>
-    <xacro:drive_wheel prefix="left" y_reflect="1"/>
-    <xacro:drive_wheel prefix="right" y_reflect="-1"/>
-    <!-- CASTER WHEEL (Rear Balance) -->
-    <link name="caster_wheel">
-        <visual>
-            <geometry>
-                <sphere radius="0.08"/>
-            </geometry>
-            <material name="black"/>
-        </visual>
-        <collision>
-            <geometry>
-                <sphere radius="0.08"/>
-            </geometry>
-        </collision>
-        <inertial>
-            <mass value="2.0"/>
-            <inertia ixx="0.005" ixy="0" ixz="0" iyy="0.005" iyz="0" izz="0.005"/>
-        </inertial>
-    </link>
-    <joint name="caster_wheel_joint" type="fixed">
-        <parent link="base_link"/>
-        <child link="caster_wheel"/>
-        <origin xyz="-0.3 0 0.08" rpy="0 0 0"/>
-    </joint>
-    <gazebo reference="caster_wheel">
-        <mu1>0.0</mu1>
-        <mu2>0.0</mu2>
-    </gazebo>
-    <!-- Gazebo Plugin for Diff Drive -->
+    <!-- Front Wheels (Low Friction for turning) -->
+    <xacro:explorer_wheel prefix="front_left" x_pos="0.18" y_pos="0.22" friction="0.01"/>
+    <xacro:explorer_wheel prefix="front_right" x_pos="0.18" y_pos="-0.22" friction="0.01"/>
+    <!-- Rear Wheels (High Friction for driving) -->
+    <xacro:explorer_wheel prefix="rear_left"  x_pos="-0.18" y_pos="0.22" friction="1.0"/>
+    <xacro:explorer_wheel prefix="rear_right" x_pos="-0.18" y_pos="-0.22" friction="1.0"/>
+    <!-- Gazebo Plugin: Diff Drive (Driving Rear Wheels) -->
     <gazebo>
         <plugin filename="gz-sim-diff-drive-system" name="gz::sim::systems::DiffDrive">
-            <left_joint>left_wheel_joint</left_joint>
-            <right_joint>right_wheel_joint</right_joint>
-            <wheel_separation>0.60</wheel_separation>
-            <wheel_radius>0.12</wheel_radius>
+            <left_joint>rear_left_wheel_joint</left_joint>
+            <right_joint>rear_right_wheel_joint</right_joint>
+            <wheel_separation>0.44</wheel_separation>
+            <wheel_radius>0.1</wheel_radius>
             <odom_publish_frequency>50</odom_publish_frequency>
             <topic>cmd_vel</topic>
@@ -187,12 +255,11 @@
             <frame_id>odom</frame_id>
             <child_frame_id>base_link</child_frame_id>
-            <covariance_x>0.0001</covariance_x>
-            <covariance_y>0.0001</covariance_y>
-            <covariance_yaw>0.01</covariance_yaw>
         </plugin>
         <plugin filename="gz-sim-joint-state-publisher-system" name="gz::sim::systems::JointStatePublisher">
             <topic>joint_states</topic>
-            <joint_name>left_wheel_joint</joint_name>
-            <joint_name>right_wheel_joint</joint_name>
+            <joint_name>rear_left_wheel_joint</joint_name>
+            <joint_name>rear_right_wheel_joint</joint_name>
+            <joint_name>front_left_wheel_joint</joint_name>
+            <joint_name>front_right_wheel_joint</joint_name>
         </plugin>
     </gazebo>
